Commit message: Added gz_ros2_control to the setup and got it working
currently hardcoded the path to the library /opt/ros/iron/lib/libgz_ros2_control-system.so
since it's not working otherwise.

File: hippo_sim/models/dynamic_arm+gripper/urdf/dynamic_arm+gripper.xacro (robot description, xacro)
@@ -79,5 +79,5 @@
         <origin xyz="0 0.05 0.10" />
         <axis xyz="0 1 0" />
-        <limit lower="0.0" upper="0.05" effort="10" velocity="1" />
+        <limit lower="-0.03" upper="0.05" effort="10" velocity="1" />
     </joint>
     <!-- Prismatic Joint for Right Finger -->
@@ -87,83 +87,33 @@
         <origin xyz="0 -0.05 0.10" />
         <axis xyz="0 -1 0" />
-        <limit lower="0.0" upper="0.05" effort="10" velocity="1" />
-        <mimic joint="finger_left_joint" multiplier="-1.0"/>
+        <limit lower="-0.03" upper="0.05" effort="10" velocity="1" />
+        <mimic joint="left_finger_joint" multiplier="1.0" />
     </joint>
-      <!-- ros2_control configuration -->
-    <ros2_control name="GripperHardware" type="system">
+    <ros2_control name="GazeboSystem" type="system">
         <hardware>
-          <plugin>fake_components/GenericSystem</plugin>
+            <plugin>gz_ros2_control/GazeboSimSystem</plugin>
         </hardware>
-        <joint name="finger_left_joint">
-          <command_interface name="position"/>
-          <state_interface name="position"/>
-          <state_interface name="velocity"/>
-          <state_interface name="effort"/>
+        <joint name="left_finger_joint">
+            <command_interface name="position" />
+            <state_interface name="position">
+                <param name="initial_value">0.02</param>
+            </state_interface>
+            <state_interface name="velocity" />
+            <state_interface name="effort" />
         </joint>
-        <joint name="finger_right_joint">
-          <command_interface name="position"/>
-          <state_interface name="position"/>
-          <state_interface name="velocity"/>
-          <state_interface name="effort"/>
+        <joint name="right_finger_joint">
+            <param name="mimic">left_finger_joint</param>
+            <param name="multiplier">1</param>
+            <command_interface name="position" />
+            <state_interface name="position" />
+            <state_interface name="velocity" />
+            <state_interface name="effort" />
         </joint>
     </ros2_control>
-          <!-- <!-1- Transmission for Left Finger -1-> -->
-  <!-- <transmission name="left_finger_transmission"> -->
-    <!-- <type>transmission_interface/SimpleTransmission</type> -->
-    <!-- <joint name="left_finger_joint"> -->
-      <!-- <hardwareInterface>hardware_interface/PositionJointInterface</hardwareInterface> -->
-    <!-- </joint> -->
-    <!-- <actuator name="left_finger_motor"> -->
-      <!-- <mechanicalReduction>1</mechanicalReduction> -->
-    <!-- </actuator> -->
-  <!-- </transmission> -->
-  <!-- <!-1- Transmission for Right Finger -1-> -->
-  <!-- <transmission name="right_finger_transmission"> -->
-    <!-- <type>transmission_interface/SimpleTransmission</type> -->
-    <!-- <joint name="right_finger_joint"> -->
-      <!-- <hardwareInterface>hardware_interface/PositionJointInterface</hardwareInterface> -->
-    <!-- </joint> -->
-    <!-- <actuator name="right_finger_motor"> -->
-      <!-- <mechanicalReduction>1</mechanicalReduction> -->
-    <!-- </actuator> -->
-  <!-- </transmission> -->
-  <!-- <!-1- ros2_control Interface -1-> -->
-  <!-- <ros2_control> -->
-    <!-- <joint name="left_finger_joint"> -->
-      <!-- <command_interface name="position"/> -->
-      <!-- <state_interface name="position"/> -->
-      <!-- <state_interface name="velocity"/> -->
-    <!-- </joint> -->
-    <!-- <joint name="right_finger_joint"> -->
-      <!-- <command_interface name="position"/> -->
-      <!-- <state_interface name="position"/> -->
-      <!-- <state_interface name="velocity"/> -->
-    <!-- </joint> -->
-  <!-- </ros2_control> -->
-    <!-- <ros2_control name="GazeboSystem" type="system"> -->
-    <!--     <hardware> -->
-    <!--         <plugin>gazebo_ros2_control/GazeboSystem</plugin> -->
-    <!--     </hardware> -->
-    <!--     <joint name="left_finger_joint"> -->
-    <!--         <command_interface name="velocity"> -->
-    <!--             <param name="min">-10</param> -->
-    <!--             <param name="max">10</param> -->
-    <!--         </command_interface> -->
-    <!--         <state_interface name="position" /> -->
-    <!--         <state_interface name="velocity" /> -->
-    <!--     </joint> -->
-    <!--     <joint name="right_finger_joint"> -->
-    <!--         <command_interface name="velocity"> -->
-    <!--             <param name="min">-10</param> -->
-    <!--             <param name="max">10</param> -->
-    <!--         </command_interface> -->
-    <!--         <state_interface name="velocity" /> -->
-    <!--         <state_interface name="position" /> -->
-    <!--     </joint> -->
-    <!-- </ros2_control> -->
-    <!-- <gazebo> -->
-    <!--     <plugin filename="libgazebo_ros2_control.so" name="gazebo_ros2_control"> -->
-    <!--         <parameters>$(find position_control)/config/controller.yaml</parameters> -->
-    <!--     </plugin> -->
-    <!-- </gazebo> -->
+    <gazebo>
+        <plugin filename="/opt/ros/iron/lib/libgz_ros2_control-system.so"
+            name="gz_ros2_control::GazeboSimROS2ControlPlugin">
+            <parameters>$(find position_control)/config/gripper_controller.yaml</parameters>
+        </plugin>
+    </gazebo>
 </robot>
