Commit message: Added an object, an arm and a rack to the simulation
Fixed the position of the Apriltags so that they are on the rack instead
of in the air

File: hippo_sim/models/bluerov/urdf/bluerov.xacro (robot description, xacro)
@@ -6,4 +6,7 @@
     <xacro:include filename="$(find hippo_sim)/models/hippo3/urdf/clamp_macro.xacro" />
     <xacro:include filename="$(find hippo_sim)/models/camera/urdf/camera_macro.xacro" />
+    <!-- <xacro:include filename="$(find hippo_sim)/models/static_arm/urdf/static_arm.xacro" /> -->
+    <xacro:include
+        filename="$(find hippo_sim)/models/dynamic_arm+gripper/urdf/dynamic_arm+gripper.xacro" />
     <xacro:property name="thruster_xy" value="${thruster_r / 2**0.5}" />
     <gazebo>
@@ -55,4 +58,9 @@
             rpy="${front_camera_orientation}" />
     </xacro:if>
+    <joint name="arm_joint" type="fixed">
+        <parent link="base_link" />
+        <child link="arm_link" />
+        <origin xyz="0 0 -0.1" rpy="0 1.57 0" />
+    </joint>
     <gazebo>
         <plugin filename="buoyancy" name="hippo_gz_plugins::buoyancy">

File: hippo_sim/models/rack/urdf/rack.xacro (robot description, xacro)
@@ -1,4 +1,4 @@
 <?xml version="1.0"?>
-<robot xmlns:xacro="http://www.ros.org/wiki/xacro" name="pool">
+<robot xmlns:xacro="http://www.ros.org/wiki/xacro" name="rack">
     <xacro:include filename="$(find hippo_sim)/models/common/urdf/common.xacro" />
     <gazebo>
@@ -6,17 +6,21 @@
     </gazebo>
     <link name="base_link">
-        <xacro:zero_inertia />
         <visual>
             <geometry>
-                <mesh filename="$(find hippo_sim)/models/pool/meshes/pool.dae" />
+                <mesh filename="$(find hippo_sim)/models/rack/meshes/rack.dae" />
             </geometry>
         </visual>
         <collision>
             <geometry>
-                <mesh filename="$(find hippo_sim)/models/pool/meshes/pool.dae" />
+                    <mesh filename="$(find hippo_sim)/models/rack/meshes/rack.dae" />
             </geometry>
         </collision>
+        <inertial>
+          <mass value="10"/>
+          <origin xyz="0 0 0"/>
+          <inertia ixx="0.1" ixy="0" ixz="0" iyy="0.1" iyz="0" izz="0.1"/>
+        </inertial>
     </link>
-    <gazebo reference="base_link">
+    <gazebo reference="rack">
         <visual>
             <material>

Commit message: Added the newton_subsea_gripper and a new test rack
Adjusted the Apriltags to still be visible with the new rack

File: hippo_sim/models/bluerov/urdf/bluerov.xacro (robot description, xacro)
@@ -7,6 +7,8 @@
     <xacro:include filename="$(find hippo_sim)/models/camera/urdf/camera_macro.xacro" />
     <!-- <xacro:include filename="$(find hippo_sim)/models/static_arm/urdf/static_arm.xacro" /> -->
+    <!-- <xacro:include -->
+    <!--     filename="$(find hippo_sim)/models/dynamic_arm+gripper/urdf/dynamic_arm+gripper.xacro" /> -->
     <xacro:include
-        filename="$(find hippo_sim)/models/dynamic_arm+gripper/urdf/dynamic_arm+gripper.xacro" />
+        filename="$(find hippo_sim)/models/newton_subsea_gripper/urdf/newton_subsea_gripper.xacro" />
     <xacro:property name="thruster_xy" value="${thruster_r / 2**0.5}" />
     <gazebo>
@@ -61,5 +63,6 @@
         <parent link="base_link" />
         <child link="arm_link" />
-        <origin xyz="0 0 -0.1" rpy="0 1.57 0" />
+        <origin xyz="0 0.0 -0.12" rpy="0 -1.57 0" />
+        <!-- <origin xyz="0 0 0" rpy="0 0 0" /> -->
     </joint>
     <gazebo>

File: hippo_sim/models/rack/urdf/rack.xacro (robot description, xacro)
@@ -8,16 +8,21 @@
         <visual>
             <geometry>
-                <mesh filename="$(find hippo_sim)/models/rack/meshes/rack.dae" />
+                <mesh filename="$(find hippo_sim)/models/rack/meshes/rack_v2.stl" />
+                <!-- <mesh filename="/home/yuna/master_thesis/parts/rack_v2.stl" /> -->
             </geometry>
+            <material name="gray">
+                <color rgba="0.5 0.5 0.5 1" />
+            </material>
         </visual>
         <collision>
             <geometry>
-                    <mesh filename="$(find hippo_sim)/models/rack/meshes/rack.dae" />
+                <mesh filename="$(find hippo_sim)/models/rack/meshes/rack_v2.stl" />
+                <!-- <mesh filename="/home/yuna/master_thesis/parts/rack_v2.stl" /> -->
             </geometry>
         </collision>
         <inertial>
-          <mass value="10"/>
-          <origin xyz="0 0 0"/>
-          <inertia ixx="0.1" ixy="0" ixz="0" iyy="0.1" iyz="0" izz="0.1"/>
+            <mass value="10" />
+            <origin xyz="0 0 0" />
+            <inertia ixx="0.1" ixy="0" ixz="0" iyy="0.1" iyz="0" izz="0.1" />
         </inertial>
     </link>

File: hippo_sim/models/test_object/urdf/test_object.xacro (robot description, xacro)
@@ -4,6 +4,5 @@
         <visual>
             <geometry>
-                <cylinder length="0.1" radius="0.04" />
-                <!-- <mesh filename="$(find hippo_sim)/models/test_object/meshes/cylinder.dae" /> -->
+                <cylinder length="0.1" radius="0.02" />
             </geometry>
             <material name="purple">
@@ -13,10 +12,9 @@
         <collision>
             <geometry>
-                <cylinder length="0.1" radius="0.04" />
-                <!-- <mesh filename="$(find hippo_sim)/models/test_object/meshes/cylinder.dae" /> -->
+                <cylinder length="0.1" radius="0.02" />
             </geometry>
         </collision>
         <inertial>
-            <mass value="0.01" />
+            <mass value="0.001" />
             <origin xyz="0 0 0" />
             <inertia ixx="0.1" ixy="0" ixz="0" iyy="0.1" iyz="0" izz="0.1" />
